File: IO4-IR-Detector-GBunza-Fingers.brd (EAGLE design)
At the start: 96.5 x 100 mm, 52 parts, among them J1 0.100, J10 0.100, J11 0.100, J12 0.100, J13 0.100, J14 0.100, J15 0.100, J16 0.100, J2 0.100, J3 0.100, J4 0.100, J5 0.100, J6 0.100, J7 0.100, J8 0.100, J9 0.100

Commit message: Version 1.3
Parts:
- moved U$1 24.1 mm to (2.54, 73.7)
- moved U$2 24.1 mm to (94.0, 73.7)
- moved T.DETECTED 12.4 mm to (6.10, 62.4)
- moved T.DETECTED10 12.4 mm to (54.4, 62.4)
- moved T.DETECTED13 12.4 mm to (78.5, 62.4)
- moved T.DETECTED15 12.4 mm to (90.6, 62.4)
- moved T.DETECTED2 12.4 mm to (18.2, 62.4)
- moved T.DETECTED4 12.4 mm to (30.2, 62.4)
- moved T.DETECTED7 12.4 mm to (42.3, 62.4)
- moved T.DETECTED8 12.4 mm to (66.4, 62.4)
- moved T.AMBIENT1 11.4 mm to (2.79, 31.1)
- moved T.AMBIENT11 11.4 mm to (51.1, 31.1)
- moved T.AMBIENT12 11.4 mm to (75.2, 31.1)
- moved T.AMBIENT14 11.4 mm to (87.2, 31.1)
- moved T.AMBIENT3 11.4 mm to (14.9, 31.1)
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Routing:
- net N$62: track 22.5 -> 21.5 mm
- net N$6: track 22.5 -> 21.5 mm
- net N$54: track 22.5 -> 21.5 mm
- net N$42: track 22.5 -> 21.5 mm
- net N$34: track 22.5 -> 21.5 mm
- net N$30: track 22.5 -> 21.5 mm
- net N$18: track 22.5 -> 21.5 mm
- net N$14: track 22.5 -> 21.5 mm
- net N$7: track 27.3 -> 26.3 mm
- net N$63: track 27.3 -> 26.3 mm
- net N$55: track 27.3 -> 26.3 mm
- net N$43: track 27.3 -> 26.3 mm
- net N$35: track 27.3 -> 26.3 mm
- net N$31: track 27.3 -> 26.3 mm
- net N$19: track 27.3 -> 26.3 mm
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Other:
- board size 96.5 x 100 mm -> 102.9 x 76.2 mm
- board text added: "For GBunza Passive IR Detector"
- board text added: "HO Midpoint N Track"
- board text added: "Track N Midpoint HO"
- board text added: "V-score"
- board text added: "WAYWAYWAY"
- board text added: "v1.3 2024.01"
- board text removed: "For GBunza Detector"
- board text removed: "JLCJLCJLCJLC"
- board text removed: "v1.2 2022.03"
